File: apu-csk-motherboard/apu-csk-motherboard.sch (EAGLE design)
At the start: 22 parts, among them U1 DS3231M+TRL

Commit message: Prototype Board for revision
Parts:
- added U$1, U$2: DIO_PMEG4030ER,115, apu-csk-motherboard:DIO_PMEG4030ER,115
- LAUNCH-SW-CN: device TSW-104-05-G-T:TSW-104-05-G-T -> apu-csk-motherboard:TSW-104-05-G-T
- R2, R3: device RMCF0805JT10K0:RMCF0805JT10K0 -> apu-csk-motherboard:RMCF0805JT10K0
Connections:
- new net FPGA3.3: PL2.3V3@4, U$1.CATHODE
- new net UC3.3: FEATHER1-16.3.3V@T15, U$2.CATHODE
- net 3.3V: now also H2.VCC_SYS@27, H2.VCC_SYS@28, U$1.ANODE, U$2.ANODE; no longer FEATHER1-16.3.3V@T15, PL2.3V3@4
- net GND: no longer H2.AGND@31
Changed lines of the file:
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@@
 <part name="SD-2" library="apu-csk-motherboard" deviceset="503182-1852" device=""/>
 <part name="AUTHENTICATION-CHIP" library="apu-csk-motherboard" deviceset="ATECC608A-SSHDA-B" device=""/>
-<part name="LAUNCH-SW-CN" library="TSW-104-05-G-T" deviceset="TSW-104-05-G-T" device=""/>
+<part name="LAUNCH-SW-CN" library="apu-csk-motherboard" deviceset="TSW-104-05-G-T" device=""/>
 <part name="TEMP-SENSE1" library="apu-csk-motherboard" deviceset="DS18B20" device=""/>
 <part name="TEMP-SENSE2" library="apu-csk-motherboard" deviceset="DS18B20" device=""/>
@@
 <part name="U1" library="apu-csk-motherboard" deviceset="DS3231M+TRL" device=""/>
 <part name="BT1" library="apu-csk-motherboard" deviceset="BK-890" device=""/>
-<part name="R2" library="RMCF0805JT10K0" deviceset="RMCF0805JT10K0" device=""/>
-<part name="R3" library="RMCF0805JT10K0" deviceset="RMCF0805JT10K0" device=""/>
+<part name="R2" library="apu-csk-motherboard" deviceset="RMCF0805JT10K0" device=""/>
+<part name="R3" library="apu-csk-motherboard" deviceset="RMCF0805JT10K0" device=""/>
+<part name="U$1" library="apu-csk-motherboard" deviceset="DIO_PMEG4030ER,115" device=""/>
+<part name="U$2" library="apu-csk-motherboard" deviceset="DIO_PMEG4030ER,115" device=""/>
 </parts>
 <sheets>
@@
 <attribute name="VALUE" x="182.886640625" y="78.73003125" size="2.54331875" layer="96" rot="R90"/>
 </instance>
+<instance part="U$1" gate="G$1" x="116.84" y="180.34" smashed="yes"/>
+<instance part="U$2" gate="G$1" x="116.84" y="172.72" smashed="yes"/>
 </instances>
 <busses>
@@
 </segment>
 <segment>
-<pinref part="H2" gate="G$1" pin="AGND@31"/>
-<wire x1="12.7" y1="40.64" x2="25.4" y2="40.64" width="0.1524" layer="91"/>
-<label x="12.7" y="40.64" size="1.778" layer="95"/>
-</segment>
-<segment>
 <pinref part="H2" gate="G$1" pin="DGND@32"/>
 <wire x1="73.66" y1="40.64" x2="60.96" y2="40.64" width="0.1524" layer="91"/>
@@
 <net name="3.3V" class="0">
 <segment>
-<pinref part="PL2" gate="G$1" pin="3V3@4"/>
-<wire x1="139.7" y1="154.94" x2="129.54" y2="154.94" width="0.1524" layer="91"/>
-<label x="139.7" y="154.94" size="1.778" layer="95" rot="MR0"/>
-</segment>
-<segment>
-<wire x1="157.48" y1="119.38" x2="167.64" y2="119.38" width="0.1524" layer="91"/>
-<label x="157.48" y="119.38" size="1.778" layer="95"/>
-<pinref part="FEATHER1" gate="-16" pin="3.3V@T15"/>
-</segment>
-<segment>
 <pinref part="SD-2" gate="G$1" pin="VDD"/>
 <wire x1="210.82" y1="129.54" x2="220.98" y2="129.54" width="0.1524" layer="91"/>
@@
 <wire x1="177.8" y1="96.52" x2="177.8" y2="101.6" width="0.1524" layer="91"/>
 <label x="177.8" y="99.06" size="1.778" layer="95" rot="R90"/>
+</segment>
+<segment>
+<pinref part="H2" gate="G$1" pin="VCC_SYS@27"/>
+<wire x1="25.4" y1="45.72" x2="12.7" y2="45.72" width="0.1524" layer="91"/>
+<label x="12.7" y="45.72" size="1.778" layer="95"/>
+</segment>
+<segment>
+<pinref part="H2" gate="G$1" pin="VCC_SYS@28"/>
+<wire x1="60.96" y1="45.72" x2="73.66" y2="45.72" width="0.1524" layer="91"/>
+<label x="73.66" y="45.72" size="1.778" layer="95" rot="MR0"/>
+</segment>
+<segment>
+<pinref part="U$1" gate="G$1" pin="ANODE"/>
+<wire x1="109.22" y1="180.34" x2="101.6" y2="180.34" width="0.1524" layer="91"/>
+<label x="101.6" y="180.34" size="1.778" layer="95"/>
+</segment>
+<segment>
+<pinref part="U$2" gate="G$1" pin="ANODE"/>
+<wire x1="101.6" y1="172.72" x2="109.22" y2="172.72" width="0.1524" layer="91"/>
+<label x="101.6" y="172.72" size="1.778" layer="95"/>
 </segment>
 </net>
@@
 </segment>
 </net>
+<net name="UC3.3" class="0">
+<segment>
+<pinref part="U$2" gate="G$1" pin="CATHODE"/>
+<wire x1="124.46" y1="172.72" x2="129.54" y2="172.72" width="0.1524" layer="91"/>
+<label x="129.54" y="172.72" size="1.778" layer="95" rot="MR0"/>
+</segment>
+<segment>
+<pinref part="FEATHER1" gate="-16" pin="3.3V@T15"/>
+<wire x1="154.94" y1="119.38" x2="167.64" y2="119.38" width="0.1524" layer="91"/>
+<label x="154.94" y="119.38" size="1.778" layer="95"/>
+</segment>
+</net>
+<net name="FPGA3.3" class="0">
+<segment>
+<pinref part="PL2" gate="G$1" pin="3V3@4"/>
+<wire x1="139.7" y1="154.94" x2="129.54" y2="154.94" width="0.1524" layer="91"/>
+<label x="139.7" y="154.94" size="1.778" layer="95"/>
+</segment>
+<segment>
+<pinref part="U$1" gate="G$1" pin="CATHODE"/>
+<wire x1="124.46" y1="180.34" x2="129.54" y2="180.34" width="0.1524" layer="91"/>
+<label x="129.54" y="180.34" size="1.778" layer="95" rot="MR0"/>
+</segment>
+</net>

Commit message: JR and Nathanael Review
Parts:
- added C1: 08053C104KAT2A, apu-csk-motherboard:08053C104KAT2A
- added C2: 08053C105KAT2A, apu-csk-motherboard:08053C105KAT2A
Connections:
- net 3.3V: now also C1.1, C2.1
- net GND: now also C1.2, C2.2
Changed lines of the file:
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@@
 <part name="U$1" library="apu-csk-motherboard" deviceset="DIO_PMEG4030ER,115" device=""/>
 <part name="U$2" library="apu-csk-motherboard" deviceset="DIO_PMEG4030ER,115" device=""/>
+<part name="C1" library="apu-csk-motherboard" deviceset="08053C104KAT2A" device=""/>
+<part name="C2" library="apu-csk-motherboard" deviceset="08053C105KAT2A" device=""/>
 </parts>
 <sheets>
@@
 <pinref part="PL2" gate="G$1" pin="3V3@4"/>
 <wire x1="139.7" y1="154.94" x2="129.54" y2="154.94" width="0.1524" layer="91"/>
-<label x="139.7" y="154.94" size="1.778" layer="95"/>
+<label x="139.7" y="154.94" size="1.778" layer="95" rot="MR0"/>
 </segment>
 <segment>
@@
 <attribute name="VALUE" x="121.92" y="105.41" size="1.778" layer="96" rot="R270"/>
 </instance>
+<instance part="C1" gate="G$1" x="142.24" y="114.3" smashed="yes" rot="R270">
+<attribute name="NAME" x="146.05093125" y="114.3" size="1.77843125" layer="95" rot="R270"/>
+<attribute name="VALUE" x="137.15151875" y="114.3" size="1.78096875" layer="96" rot="R270"/>
+</instance>
+<instance part="C2" gate="G$1" x="154.94" y="114.3" smashed="yes" rot="R270">
+<attribute name="NAME" x="158.75093125" y="114.3" size="1.77843125" layer="95" rot="R270"/>
+<attribute name="VALUE" x="149.85151875" y="114.3" size="1.78096875" layer="96" rot="R270"/>
+</instance>
 </instances>
 <busses>
@@
 <label x="119.38" y="93.98" size="1.778" layer="95"/>
 </segment>
+<segment>
+<pinref part="C1" gate="G$1" pin="2"/>
+<wire x1="142.24" y1="109.22" x2="142.24" y2="104.14" width="0.1524" layer="91"/>
+<label x="142.24" y="104.14" size="1.778" layer="95" rot="R90"/>
+</segment>
+<segment>
+<pinref part="C2" gate="G$1" pin="2"/>
+<wire x1="154.94" y1="109.22" x2="154.94" y2="104.14" width="0.1524" layer="91"/>
+<label x="154.94" y="104.14" size="1.778" layer="95" rot="R90"/>
+</segment>
 </net>
 <net name="3.3V" class="0">
@@
 <segment>
 <pinref part="U1" gate="A" pin="VCC"/>
-<wire x1="114.3" y1="119.38" x2="124.46" y2="119.38" width="0.1524" layer="91"/>
-<label x="124.46" y="119.38" size="1.778" layer="95"/>
-</segment>
-</net>
+<wire x1="114.3" y1="119.38" x2="142.24" y2="119.38" width="0.1524" layer="91"/>
+<label x="160.02" y="119.38" size="1.778" layer="95"/>
+<pinref part="C2" gate="G$1" pin="1"/>
+<wire x1="142.24" y1="119.38" x2="154.94" y2="119.38" width="0.1524" layer="91"/>
+<wire x1="154.94" y1="119.38" x2="160.02" y2="119.38" width="0.1524" layer="91"/>
+<wire x1="154.94" y1="116.84" x2="154.94" y2="119.38" width="0.1524" layer="91"/>
+<junction x="154.94" y="119.38"/>
+<pinref part="C1" gate="G$1" pin="1"/>
+<wire x1="142.24" y1="116.84" x2="142.24" y2="119.38" width="0.1524" layer="91"/>
+<junction x="142.24" y="119.38"/>
+</segment>
+</net>

Commit message: Almost done
Parts:
- removed AUTHENTICATION-CHIP: ATECC608A-SSHDA-B, apu-csk-motherboard:ATECC608A-SSHDA-B
- removed LAUNCH-SW-CN: TSW-104-05-G-T, apu-csk-motherboard:TSW-104-05-G-T
- removed TEMP-SENSE4: DS18B20, apu-csk-motherboard:DS18B20
- added J2: TSW-108-05-G-S, apu-csk-motherboard:TSW-108-05-G-S
- added P1: ATECC608A-SSHDA-B, apu-csk-motherboard:ATECC608A-SSHDA-B
- added S1: 463092691402, apu-csk-motherboard:463092691402
- added T1: DS18B20, apu-csk-motherboard:DS18B20
- renumbered TEMP-SENSE1 to T2, TEMP-SENSE2 to T3, TEMP-SENSE3 to T4, U$1 to B1, U$2 to B2
Connections:
- removed net LSW-1-C: LAUNCH-SW-CNG$2.03, PL2.B1@30
- removed net LSW-1-NC: LAUNCH-SW-CNG$1.01, PL2.N1@14
- removed net LSW-1-NO: LAUNCH-SW-CNG$1.02, PL2.G3@22
- removed net LSW-2-C: LAUNCH-SW-CNG$2.06, PL2.A2@32
- removed net LSW-2-NC: LAUNCH-SW-CNG$1.04, PL2.L1@16
- removed net LSW-2-NO: LAUNCH-SW-CNG$1.05, PL2.F3@24
- removed net LSW-3-C: LAUNCH-SW-CNG$2.09, PL2.C4@34
- removed net LSW-3-NC: LAUNCH-SW-CNG$1.07, PL2.J3@18
- removed net LSW-3-NO: LAUNCH-SW-CNG$1.08, PL2.D1@26
- removed net LSW-4-C: LAUNCH-SW-CNG$2.12, PL2.C5@36
- removed net LSW-4-NC: LAUNCH-SW-CNG$1.10, PL2.H3@20
- removed net LSW-4-NO: LAUNCH-SW-CNG$1.11, PL2.D3@28
- new net LS_C: H2.S5@43, H2.S5@44, J2.01
- new net LS_NC: H2.S1@35, H2.S1@36, J2.08
- new net N$3: J2.02, J2.03
- new net N$4: J2.04, J2.05
- new net N$5: J2.06, J2.07
- new net RBF_C: H2.S4@41, H2.S4@42, S1.COM
- new net RBF_NC: H2.S0@33, H2.S0@34, S1.NC
- net 3.3V: now also P1.VCC, T1.VDD; no longer AUTHENTICATION-CHIP.VCC, TEMP-SENSE4.VDD
- net DQ-TEMP: now also T1.DQ; no longer TEMP-SENSE4.DQ
- net GND: now also P1.GND, T1.GND; no longer AUTHENTICATION-CHIP.GND, TEMP-SENSE4.GND
- net SCL: now also P1.SCL; no longer AUTHENTICATION-CHIP.SCL
- net SDA: now also P1.SDA; no longer AUTHENTICATION-CHIP.SDA
