File: apu-csk-motherboard/apu-csk-motherboard.brd (EAGLE design)
At the start: 90.2 x 95.9 mm, 22 parts, among them U1 DS3231M+TRL

Commit message: Prototype Board for revision
Parts:
- added U$1, U$2: DIO_PMEG4030ER,115, apu-csk-motherboard:DIO_PMEG4030ER,115
- LAUNCH-SW-CN: device TSW-104-05-G-T:SAMTEC_TSW-104-05-G-T -> apu-csk-motherboard:SAMTEC_TSW-104-05-G-T
- R2, R3: device RMCF0805JT10K0:RESC2012X65N -> apu-csk-motherboard:RESC2012X65N
- moved AUTHENTICATION-CHIP 1.12 mm to (54.0, 48.5), turned to 270 degrees
- moved LAUNCH-SW-CN 1.00 mm to (40.0, 46.0)
Connections:
- new net FPGA3.3: PL2.4, U$1.1
- new net UC3.3: FEATHER1.T15, U$2.1
- net 3.3V: now also H2.27, H2.28, U$1.2, U$2.2; no longer FEATHER1.T15, PL2.4
- net GND: no longer H2.31
Routing:
- net 3.3V: track 0.00 -> 468.4 mm
- net GND: track 0.00 -> 407.8 mm, vias 0 -> 5
- net DQ-TEMP: track 0.00 -> 290.3 mm
- net SCL: track 0.00 -> 152.7 mm, vias 0 -> 3
- net SDA: track 0.00 -> 144.7 mm, vias 0 -> 4
- net COPI: track 0.00 -> 120.8 mm, vias 0 -> 2
- net SCK: track 0.00 -> 115.5 mm, vias 0 -> 4
- net USER0: track 0.00 -> 104.6 mm
- net FE_V_USB: track 0.00 -> 98.6 mm, vias 0 -> 1
- net CIPO: track 0.00 -> 97.8 mm, vias 0 -> 4
- net USER9: track 0.00 -> 91.1 mm
- net FE_IO2: track 0.00 -> 88.2 mm, vias 0 -> 1
- net USER1: track 0.00 -> 87.6 mm, vias 0 -> 1
- net CS-SD-1: track 0.00 -> 87.6 mm, vias 0 -> 1
- net FE_IO10: track 0.00 -> 76.6 mm
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
Commit message: JR and Nathanael Review
Parts:
- added C1: 08053C104KAT2A, apu-csk-motherboard:CAPC2012X94N
- added C2: 08053C105KAT2A, apu-csk-motherboard:CAPC2012X94N
- turned AUTHENTICATION-CHIP to 90 degrees
Connections:
- net 3.3V: now also C1.1, C2.1
- net GND: now also C1.2, C2.2
Routing:
- net 3.3V: track 468.4 -> 407.2 mm, vias 0 -> 3
- net SCK: track 115.5 -> 162.1 mm
- net FE_V_USB: track 98.6 -> 54.1 mm, vias 1 -> 0
- net FE_IO2: track 88.2 -> 50.9 mm, vias 1 -> 0
- net GND: track 407.8 -> 443.7 mm, vias 5 -> 4
- net USER0: track 104.6 -> 73.3 mm, vias 0 -> 1
- net USER9: track 91.1 -> 64.1 mm, vias 0 -> 3
- net CS-SD-1: track 87.6 -> 63.4 mm, vias 1 -> 2
- net LSW-2-C: track 29.2 -> 52.7 mm, vias 1 -> 0
- net SCL: track 152.7 -> 130.1 mm, vias 3 -> 2
- net USER1: track 87.6 -> 67.6 mm, vias 1 -> 2
- net CS-SD-2: track 66.1 -> 84.3 mm, vias 3 -> 1
- net FE_IO10: track 76.6 -> 61.4 mm
- net SDA: track 144.7 -> 130.8 mm, vias 4 -> 3
- net LSW-3-NC: track 45.1 -> 57.8 mm, vias 1 -> 0
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
Commit message: Almost done
Parts:
- removed AUTHENTICATION-CHIP: ATECC608A-SSHDA-B, apu-csk-motherboard:SOIC127P600X175-8N
- removed LAUNCH-SW-CN: TSW-104-05-G-T, apu-csk-motherboard:SAMTEC_TSW-104-05-G-T
- added J2: TSW-108-05-G-S, apu-csk-motherboard:SAMTEC_TSW-108-05-G-S
- added P1: ATECC608A-SSHDA-B, apu-csk-motherboard:SOIC127P600X175-8N
- added S1: 463092691402, apu-csk-motherboard:463092691402
- renumbered TEMP-SENSE1 to T1, TEMP-SENSE2 to T2, TEMP-SENSE3 to T3, TEMP-SENSE4 to T4, U$1 to B1, U$2 to B2
Connections:
- removed net LSW-1-C: LAUNCH-SW-CN.03, PL2.30
- removed net LSW-1-NC: LAUNCH-SW-CN.01, PL2.14
- removed net LSW-1-NO: LAUNCH-SW-CN.02, PL2.22
- removed net LSW-2-C: LAUNCH-SW-CN.06, PL2.32
- removed net LSW-2-NC: LAUNCH-SW-CN.04, PL2.16
- removed net LSW-2-NO: LAUNCH-SW-CN.05, PL2.24
- removed net LSW-3-C: LAUNCH-SW-CN.09, PL2.34
- removed net LSW-3-NC: LAUNCH-SW-CN.07, PL2.18
- removed net LSW-3-NO: LAUNCH-SW-CN.08, PL2.26
- removed net LSW-4-C: LAUNCH-SW-CN.12, PL2.36
- removed net LSW-4-NC: LAUNCH-SW-CN.10, PL2.20
- removed net LSW-4-NO: LAUNCH-SW-CN.11, PL2.28
- new net LS_C: H2.43, H2.44, J2.01
- new net LS_NC: H2.35, H2.36, J2.08
- new net N$3: J2.02, J2.03
- new net N$4: J2.04, J2.05
- new net N$5: J2.06, J2.07
- new net RBF_C: H2.41, H2.42, S1.1
- new net RBF_NC: H2.33, H2.34, S1.3
- net 3.3V: now also P1.8; no longer AUTHENTICATION-CHIP.8
- net GND: now also P1.4; no longer AUTHENTICATION-CHIP.4
- net SCL: now also P1.6; no longer AUTHENTICATION-CHIP.6
- net SDA: now also P1.5; no longer AUTHENTICATION-CHIP.5
Routing:
- net LSW-3-NC: track 57.8 -> 0.00 mm
- net LSW-2-C: track 52.7 -> 0.00 mm
- net LSW-4-NC: track 52.0 -> 0.00 mm, vias 1 -> 0
- net LS_C: track 0.00 -> 51.9 mm, vias 0 -> 1
- net USER4: track 71.0 -> 120.7 mm, vias 1 -> 0
- net LS_NC: track 0.00 -> 45.5 mm
- net LSW-2-NC: track 41.9 -> 0.00 mm, vias 1 -> 0
- net LSW-1-NC: track 40.8 -> 0.00 mm
- net RBF_NC: track 0.00 -> 38.7 mm
- net USER0: track 73.3 -> 109.4 mm
- net 3.3V: track 407.2 -> 442.9 mm, vias 3 -> 4
- net LSW-4-NO: track 35.6 -> 0.00 mm
- net LSW-3-NO: track 35.4 -> 0.00 mm
- net LSW-1-NO: track 35.2 -> 0.00 mm
- net LSW-2-NO: track 35.1 -> 0.00 mm
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
Commit message: JR to review
Parts:
- moved S1 1.00 mm to (67.0, 62.0)
Routing:
- net USER11: track 90.0 -> 59.7 mm, vias 0 -> 2
- net 3.3V: track 442.9 -> 470.9 mm
- net SCK: track 145.0 -> 118.8 mm
- net GND: track 420.2 -> 439.0 mm
- net SDA: track 128.8 -> 112.2 mm, vias 2 -> 3
- net FE_IO11: track 67.6 -> 51.7 mm
- net USER4: track 120.7 -> 106.1 mm
- net USER2: track 81.9 -> 96.3 mm, vias 1 -> 0
- net CS-SD-2: track 78.5 -> 91.9 mm, vias 1 -> 0
- net FE_IO2: track 63.1 -> 50.9 mm, vias 0 -> 1
- net FE_EN: track 57.0 -> 69.1 mm
- net USER1: track 84.1 -> 74.5 mm
- net CS-FRAM: track 36.8 -> 30.3 mm, vias 0 -> 1
- net UC3.3: track 42.0 -> 48.2 mm
- net FE_IO10: track 51.2 -> 56.4 mm, vias 2 -> 1
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
Commit message: RBF Placement
Parts:
- moved S1 1.00 mm to (66.0, 62.0)
Routing:
- net USER11: track 59.7 -> 90.0 mm, vias 2 -> 0
- net 3.3V: track 470.9 -> 442.9 mm
- net SCK: track 118.8 -> 145.0 mm
- net GND: track 439.0 -> 420.2 mm
- net SDA: track 112.2 -> 128.8 mm, vias 3 -> 2
- net FE_IO11: track 51.7 -> 67.6 mm
- net USER4: track 106.1 -> 120.7 mm
- net USER2: track 96.3 -> 81.9 mm, vias 0 -> 1
- net CS-SD-2: track 91.9 -> 78.5 mm, vias 0 -> 1
- net FE_IO2: track 50.9 -> 63.1 mm, vias 1 -> 0
- net FE_EN: track 69.1 -> 57.0 mm
- net USER1: track 74.5 -> 84.1 mm
- net CS-FRAM: track 30.3 -> 36.8 mm, vias 1 -> 0
- net UC3.3: track 48.2 -> 42.0 mm
- net FE_IO10: track 56.4 -> 51.2 mm, vias 1 -> 2
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